File: 0021_Current_Module_ACS712.kicad_sch (KiCad schematic)
At the start: 6 parts, among them J1 Screw_Terminal_01x02, U1 ACS712xLCTR-20A

Commit message: Add files via upload
Parts:
- added D1: LED, LED_SMD:LED_0805_2012Metric, symbol Device:LED
- added R2: 470R, Resistor_SMD:R_0805_2012Metric, symbol Device:R
- added U3: ~, Moduler_:pin_header, symbol moduler_pin:air
- C1, C2, C3: footprint (none) -> Capacitor_SMD:C_0805_2012Metric
- J1: footprint (none) -> barriyer:barriyer_7.62
- R1: footprint (none) -> Resistor_SMD:R_0805_2012Metric
Connections:
- net GND: now also D1.1 (K), U3.9
- net SIG: now also U3.12
- net +5V: now reaches C2.1, C3.1, U1.8 (VCC)
- net +5V: now also R2.2, U3.7
- net at U1.1 (IP+), U1.2 (IP+): now also J1.2 (Pin_2); no longer J1.1 (Pin_1)
- net at U1.3 (IP-), U1.4 (IP-): now also J1.1 (Pin_1); no longer J1.2 (Pin_2)
- new net: D1.2 (A), R2.1
- no-connect marks 0 -> 15
Other:
- note added: "AIR PIN"
- note added: "SENSOR"
- moved on the sheet: C1, C2, C3, R1, U1
